File: electrical design/layer4/layer4.kicad_pcb (KiCad board)
At the start: 2 copper layers, 0 parts

Commit message: finalise l4 sch, start draft of l4 pcb
Parts:
- added C1: 0.1µF, Capacitor_SMD:C_0603_1608Metric, F.Cu at (112.0, 74.0)
- added C10: 0.1µF, Capacitor_SMD:C_0603_1608Metric, F.Cu at (89.0, 129.5)
- added C11: 0.1µF, Capacitor_SMD:C_0603_1608Metric, F.Cu at (95.7, 134.7)
- added C12: 0.1µF, Capacitor_SMD:C_0603_1608Metric, F.Cu at (103.6, 138.0)
- added C13: 0.1µF, Capacitor_SMD:C_0603_1608Metric, F.Cu at (112.0, 139.1)
- added C14: 0.1µF, Capacitor_SMD:C_0603_1608Metric, F.Cu at (120.4, 138.0)
- added C15: 0.1µF, Capacitor_SMD:C_0603_1608Metric, F.Cu at (128.3, 134.7)
- added C16: 0.1µF, Capacitor_SMD:C_0603_1608Metric, F.Cu at (135.0, 129.5)
- added C17: 0.1µF, Capacitor_SMD:C_0603_1608Metric, F.Cu at (140.2, 122.8)
- added C18: 0.1µF, Capacitor_SMD:C_0603_1608Metric, F.Cu at (143.4, 115.0)
- added C19: 0.1µF, Capacitor_SMD:C_0603_1608Metric, F.Cu at (144.5, 106.6)
- added C2: 0.1µF, Capacitor_SMD:C_0603_1608Metric, F.Cu at (103.6, 75.1)
- added C20: 0.1µF, Capacitor_SMD:C_0603_1608Metric, F.Cu at (143.4, 98.1)
- added C21: 0.1µF, Capacitor_SMD:C_0603_1608Metric, F.Cu at (140.2, 90.3)
- added C22: 0.1µF, Capacitor_SMD:C_0603_1608Metric, F.Cu at (135.0, 83.6)
- added C23: 0.1µF, Capacitor_SMD:C_0603_1608Metric, F.Cu at (128.3, 78.4)
- added C24: 0.1µF, Capacitor_SMD:C_0603_1608Metric, F.Cu at (120.4, 75.1)
- added C3: 0.1µF, Capacitor_SMD:C_0603_1608Metric, F.Cu at (95.7, 78.4)
- added C4: 0.1µF, Capacitor_SMD:C_0603_1608Metric, F.Cu at (89.0, 83.6)
- added C5: 0.1µF, Capacitor_SMD:C_0603_1608Metric, F.Cu at (83.8, 90.3)
- added C6: 0.1µF, Capacitor_SMD:C_0603_1608Metric, F.Cu at (80.6, 98.1)
- added C7: 0.1µF, Capacitor_SMD:C_0603_1608Metric, F.Cu at (79.5, 106.6)
- added C8: 0.1µF, Capacitor_SMD:C_0603_1608Metric, F.Cu at (80.6, 115.0)
- added C9: 0.1µF, Capacitor_SMD:C_0603_1608Metric, F.Cu at (83.8, 122.8)
- added D1: WS2812B, LED_SMD:LED_WS2812B_PLCC4_5.0x5.0mm_P3.2mm, F.Cu at (112.0, 68.7)
- added D10: WS2812B, LED_SMD:LED_WS2812B_PLCC4_5.0x5.0mm_P3.2mm, F.Cu at (85.2, 133.3)
- added D11: WS2812B, LED_SMD:LED_WS2812B_PLCC4_5.0x5.0mm_P3.2mm, F.Cu at (93.1, 139.3)
- added D12: WS2812B, LED_SMD:LED_WS2812B_PLCC4_5.0x5.0mm_P3.2mm, F.Cu at (102.2, 143.1)
- added D13: WS2812B, LED_SMD:LED_WS2812B_PLCC4_5.0x5.0mm_P3.2mm, F.Cu at (112.0, 144.4)
- added D14: WS2812B, LED_SMD:LED_WS2812B_PLCC4_5.0x5.0mm_P3.2mm, F.Cu at (121.8, 143.1)
- added D15: WS2812B, LED_SMD:LED_WS2812B_PLCC4_5.0x5.0mm_P3.2mm, F.Cu at (130.9, 139.3)
- added D16: WS2812B, LED_SMD:LED_WS2812B_PLCC4_5.0x5.0mm_P3.2mm, F.Cu at (138.8, 133.3)
- added D17: WS2812B, LED_SMD:LED_WS2812B_PLCC4_5.0x5.0mm_P3.2mm, F.Cu at (144.8, 125.5)
- added D18: WS2812B, LED_SMD:LED_WS2812B_PLCC4_5.0x5.0mm_P3.2mm, F.Cu at (148.6, 116.3)
- added D19: WS2812B, LED_SMD:LED_WS2812B_PLCC4_5.0x5.0mm_P3.2mm, F.Cu at (149.8, 106.6)
- added D2: WS2812B, LED_SMD:LED_WS2812B_PLCC4_5.0x5.0mm_P3.2mm, F.Cu at (102.2, 70.0)
- added D20: WS2812B, LED_SMD:LED_WS2812B_PLCC4_5.0x5.0mm_P3.2mm, F.Cu at (148.6, 96.8)
- added D21: WS2812B, LED_SMD:LED_WS2812B_PLCC4_5.0x5.0mm_P3.2mm, F.Cu at (144.8, 87.6)
- added D22: WS2812B, LED_SMD:LED_WS2812B_PLCC4_5.0x5.0mm_P3.2mm, F.Cu at (138.8, 79.8)
- added D23: WS2812B, LED_SMD:LED_WS2812B_PLCC4_5.0x5.0mm_P3.2mm, F.Cu at (130.9, 73.8)
- added D24: WS2812B, LED_SMD:LED_WS2812B_PLCC4_5.0x5.0mm_P3.2mm, F.Cu at (121.8, 70.0)
- added D3: WS2812B, LED_SMD:LED_WS2812B_PLCC4_5.0x5.0mm_P3.2mm, F.Cu at (93.1, 73.8)
- added D4: WS2812B, LED_SMD:LED_WS2812B_PLCC4_5.0x5.0mm_P3.2mm, F.Cu at (85.2, 79.8)
- added D5: WS2812B, LED_SMD:LED_WS2812B_PLCC4_5.0x5.0mm_P3.2mm, F.Cu at (79.2, 87.6)
- added D6: WS2812B, LED_SMD:LED_WS2812B_PLCC4_5.0x5.0mm_P3.2mm, F.Cu at (75.4, 96.8)
- added D7: WS2812B, LED_SMD:LED_WS2812B_PLCC4_5.0x5.0mm_P3.2mm, F.Cu at (74.2, 106.6)
- added D8: WS2812B, LED_SMD:LED_WS2812B_PLCC4_5.0x5.0mm_P3.2mm, F.Cu at (75.4, 116.3)
- added D9: WS2812B, LED_SMD:LED_WS2812B_PLCC4_5.0x5.0mm_P3.2mm, F.Cu at (79.2, 125.5)
Routing:
- added copper zone on F.Cu, net +5V
Other:
- board text added: "8076 ROBOTICS"

Commit message: production ready layer 4!
Parts:
- added J1: Conn_01x03_Male, Connector_JST:JST_SH_SM03B-SRSS-TB_1x03-1MP_P1.00mm_Horizontal, F.Cu at (137.0, 159.0)
- moved D11 9.47 mm to (88.3, 147.5), turned to 60 degrees
- moved D10 9.40 mm to (79.4, 140.6), turned to 45 degrees
- moved D12 9.39 mm to (98.8, 151.9), turned to 75 degrees
- moved D9 9.16 mm to (72.5, 131.7), turned to 30 degrees
- moved D13 9.16 mm to (110.0, 153.3), turned to 90 degrees
- moved D8 8.77 mm to (68.1, 121.2), turned to 15 degrees
- moved D14 8.77 mm to (121.2, 151.9), turned to 105 degrees
- moved C11 8.47 mm to (91.5, 142.0)
- moved C10 8.40 mm to (83.8, 136.2)
- moved C12 8.40 mm to (100.4, 145.7)
- moved D7 8.24 mm to (66.7, 110.0), turned to 0 degrees
- moved D15 8.24 mm to (131.7, 147.5), turned to 120 degrees
- moved C9 8.19 mm to (78.0, 128.5)
- moved C13 8.19 mm to (110.0, 147.0)
- moved C8 7.83 mm to (74.3, 119.6)
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Connections:
- D1 pad 4: NEOPIXELOUT -> /NEOPIXELOUT
Routing:
- net GND: track 0.00 -> 224.6 mm, vias 0 -> 25
- net /NEOPIXELOUT: track 0.00 -> 142.3 mm
- net Net-(D7-Pad2): track 0.00 -> 9.87 mm
- net Net-(D1-Pad2): track 0.00 -> 9.87 mm
- net Net-(D19-Pad2): track 0.00 -> 9.87 mm
- net Net-(D13-Pad2): track 0.00 -> 9.87 mm
- net Net-(D14-Pad2): track 0.00 -> 9.87 mm
- net Net-(D8-Pad2): track 0.00 -> 9.87 mm
- net Net-(D18-Pad2): track 0.00 -> 9.87 mm
- net Net-(D12-Pad2): track 0.00 -> 9.87 mm
- net Net-(D20-Pad2): track 0.00 -> 9.87 mm
- net Net-(D6-Pad2): track 0.00 -> 9.87 mm
- net Net-(D2-Pad2): track 0.00 -> 9.87 mm
- net Net-(D5-Pad2): track 0.00 -> 9.87 mm
- net Net-(D21-Pad2): track 0.00 -> 9.87 mm
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- added copper zone on B.Cu, net GND
Other:
- board outline added: 120 x 157.9 mm
- board text removed: "8076 ROBOTICS"
