File: electrical design/layer4/layer4.kicad_sch (KiCad schematic)
At the start: 0 parts

Commit message: finalise l4 sch, start draft of l4 pcb
Parts:
- added C1, C10, C11, C12, C13, C14, C15, C16, C17, C18, C19, C2, C20, C21, C22, C23, C24, C3, C4, C5, C6, C7, C8, C9: 0.1µF, Capacitor_SMD:C_0603_1608Metric, symbol Device:C
- added D1, D10, D11, D12, D13, D14, D15, D16, D17, D18, D19, D2, D20, D21, D22, D23, D24, D3, D4, D5, D6, D7, D8, D9: WS2812B, LED_SMD:LED_WS2812B_PLCC4_5.0x5.0mm_P3.2mm, symbol LED:WS2812B
- added J?: Conn_01x03_Male, symbol Connector:Conn_01x03_Male
Connections:
- new net: D16.2 (DOUT), D17.4 (DIN)
- new net: D15.2 (DOUT), D16.4 (DIN)
- new net: D8.2 (DOUT), D9.4 (DIN)
- new net: D7.2 (DOUT), D8.4 (DIN)
- new net: D11.2 (DOUT), D12.4 (DIN)
- new net: D10.2 (DOUT), D11.4 (DIN)
- new net: D5.2 (DOUT), D6.4 (DIN)
- new net: D4.2 (DOUT), D5.4 (DIN)
- new net: D12.2 (DOUT), D13.4 (DIN)
- new net: D19.2 (DOUT), D20.4 (DIN)
- new net: D18.2 (DOUT), D19.4 (DIN)
- new net: D22.2 (DOUT), D23.4 (DIN)
- new net: D21.2 (DOUT), D22.4 (DIN)
- new net: D14.2 (DOUT), D15.4 (DIN)
- new net: D13.2 (DOUT), D14.4 (DIN)
- new net: D6.2 (DOUT), D7.4 (DIN)
- new net: D17.2 (DOUT), D18.4 (DIN)
- new net: D20.2 (DOUT), D21.4 (DIN)
- new net: D10.4 (DIN), D9.2 (DOUT)
- new net: D2.2 (DOUT), D3.4 (DIN)
- new net: D1.2 (DOUT), D2.4 (DIN)
- new net: D3.2 (DOUT), D4.4 (DIN)
- new net: D23.2 (DOUT), D24.4 (DIN)
- new net +5V: C1.1, C10.1, C11.1, C12.1, C13.1, C14.1, C15.1, C16.1, C17.1, C18.1, C19.1, C2.1, C20.1, C21.1, C22.1, C23.1, C24.1, C3.1, C4.1, C5.1, C6.1, C7.1, C8.1, C9.1, D1.1 (VDD), D10.1 (VDD), D11.1 (VDD), D12.1 (VDD), D13.1 (VDD), D14.1 (VDD), D15.1 (VDD), D16.1 (VDD), D17.1 (VDD), D18.1 (VDD), D19.1 (VDD), D2.1 (VDD), D20.1 (VDD), D21.1 (VDD), D22.1 (VDD), D23.1 (VDD), D24.1 (VDD), D3.1 (VDD), D4.1 (VDD), D5.1 (VDD), D6.1 (VDD), D7.1 (VDD), D8.1 (VDD), D9.1 (VDD), J?.1 (Pin_1)
- new net GND: C1.2, C10.2, C11.2, C12.2, C13.2, C14.2, C15.2, C16.2, C17.2, C18.2, C19.2, C2.2, C20.2, C21.2, C22.2, C23.2, C24.2, C3.2, C4.2, C5.2, C6.2, C7.2, C8.2, C9.2, D1.3 (VSS), D10.3 (VSS), D11.3 (VSS), D12.3 (VSS), D13.3 (VSS), D14.3 (VSS), D15.3 (VSS), D16.3 (VSS), D17.3 (VSS), D18.3 (VSS), D19.3 (VSS), D2.3 (VSS), D20.3 (VSS), D21.3 (VSS), D22.3 (VSS), D23.3 (VSS), D24.3 (VSS), D3.3 (VSS), D4.3 (VSS), D5.3 (VSS), D6.3 (VSS), D7.3 (VSS), D8.3 (VSS), D9.3 (VSS), J?.2 (Pin_2)
- new net NEOPIXELOUT: D1.4 (DIN), J?.3 (Pin_3)

Commit message: almost final pcbs
Parts:
- gave numbers to parts that had none: 1
Changed lines of the file:
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@@
   (symbol (lib_id "Connector:Conn_01x03_Male") (at 30.48 151.13 0) (unit 1)
     (in_bom yes) (on_board yes) (fields_autoplaced)
-    (property "Reference" "J?" (id 0) (at 31.115 143.51 0))
+    (property "Reference" "J1" (id 0) (at 31.115 143.51 0))
     (property "Value" "Conn_01x03_Male" (id 1) (at 31.115 146.05 0))
     (property "Footprint" "" (id 2) (at 30.48 151.13 0)
@@
     )
     (path "/5a7ba987-f39e-4381-9b8f-5f907409fe0a"
-      (reference "J?") (unit 1) (value "Conn_01x03_Male") (footprint "")
-    )
-  )
+      (reference "J1") (unit 1) (value "Conn_01x03_Male") (footprint "")
+    )
+  )

Commit message: production ready layer 4!
Parts:
- J1: footprint (none) -> Connector_JST:JST_SH_SM03B-SRSS-TB_1x03-1MP_P1.00mm_Horizontal
Changed lines of the file:
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@@
   (title_block
     (title "layer 4  schematic drawing")
-    (date "2023-01-29")
-    (rev "0.3")
+    (date "2023-02-12")
+    (rev "1.0")
     (company "8076 Robotics")
   )
@@
   (symbol (lib_id "power:GND") (at 35.56 151.13 90) (unit 1)
     (in_bom yes) (on_board yes) (fields_autoplaced)
-    (property "Reference" "#PWR?" (id 0) (at 41.91 151.13 0)
+    (property "Reference" "#PWR0101" (id 0) (at 41.91 151.13 0)
       (effects (font (size 1.27 1.27)) hide)
     )
@@
     (property "Reference" "J1" (id 0) (at 31.115 143.51 0))
     (property "Value" "Conn_01x03_Male" (id 1) (at 31.115 146.05 0))
-    (property "Footprint" "" (id 2) (at 30.48 151.13 0)
+    (property "Footprint" "Connector_JST:JST_SH_SM03B-SRSS-TB_1x03-1MP_P1.00mm_Horizontal" (id 2) (at 30.48 151.13 0)
       (effects (font (size 1.27 1.27)) hide)
     )
@@
   (symbol (lib_id "power:+5V") (at 35.56 148.59 270) (unit 1)
     (in_bom yes) (on_board yes) (fields_autoplaced)
-    (property "Reference" "#PWR?" (id 0) (at 31.75 148.59 0)
+    (property "Reference" "#PWR0102" (id 0) (at 31.75 148.59 0)
       (effects (font (size 1.27 1.27)) hide)
     )
@@
     )
     (path "/54b68426-a0ca-4bb3-9290-4735fe280002"
-      (reference "#PWR?") (unit 1) (value "GND") (footprint "")
+      (reference "#PWR0101") (unit 1) (value "GND") (footprint "")
     )
     (path "/d8df21ba-053b-45ed-8e77-c5f3a40b7fd4"
-      (reference "#PWR?") (unit 1) (value "+5V") (footprint "")
+      (reference "#PWR0102") (unit 1) (value "+5V") (footprint "")
     )
     (path "/063c0627-ff19-45c9-9ddb-6bd81a0d2d41"
@@
     )
     (path "/5a7ba987-f39e-4381-9b8f-5f907409fe0a"
-      (reference "J1") (unit 1) (value "Conn_01x03_Male") (footprint "")
-    )
-  )
+      (reference "J1") (unit 1) (value "Conn_01x03_Male") (footprint "Connector_JST:JST_SH_SM03B-SRSS-TB_1x03-1MP_P1.00mm_Horizontal")
+    )
+  )
