File: electrical design/layer5/layer5.kicad_sch (KiCad schematic)
At the start: 49 parts, among them J1 Conn_01x03_Male

Commit message: rename all layer 4 files to layer 5
Other:
- title: layer 4  schematic drawing -> layer 5 schematic drawing
Changed lines of the file:
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@@
   (paper "A4")
   (title_block
-    (title "layer 4  schematic drawing")
+    (title "layer 5 schematic drawing")
     (date "2023-02-12")
     (rev "1.0")
