File: electrical design/layer1/layer1.kicad_sch (KiCad schematic)
At the start: 107 parts, among them J1 SH1.0 Female, J2 SH1.0 5P, J4 Conn_01x03_Female, J5 Conn_01x02_Female, Q1 MOSFET-NCH-FQP30N06L, Q2 MOSFET-NCH-AO3404A, SW1 SW_DPDT_x2, SW2 SW_DPDT_x2, SW3 SW_Push, U1 STM32F103C8T6, U2 CD74HC4067SM, U3 CD74HC4067SM, Y1 Crystal

Commit message: production-ready layer 1!
Parts:
- removed R33: 0.39, Resistor_SMD:R_0603_1608Metric, symbol Device:R
- added J5, J6: Conn_01x02_Male, Connector_PinHeader_2.54mm:PinHeader_1x02_P2.54mm_Vertical, symbol Connector:Conn_01x02_Male
- J3: renamed from J4; value Conn_01x03_Female -> DEBUG
- renumbered J5 to J4
Connections:
- net +5V: now also J5.1 (Pin_1)
- net GND: now also J5.2 (Pin_2)
- net VCCQ: now also J6.1 (Pin_1)
- net at C1.1, D1.2 (A), D10.2 (A)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: now also SW1.2 (B)
- net LIGHTGATE: now reaches U1.14 (PA4)
- net LIGHTGATE: now also J6.2 (Pin_2)
Changed lines of the file:
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@@
   (title_block
     (title "layer 1 schematic drawing")
-    (date "2023-02-05")
-    (rev "v0.5")
+    (date "2023-02-15")
+    (rev "v1.0")
     (company "8076 Robotics")
   )
@@
     (stroke (width 0) (type default) (color 0 0 0 0))
   )
-  (wire (pts (xy 39.37 25.4) (xy 41.91 25.4))
-    (stroke (width 0) (type default) (color 0 0 0 0))
-  )
   (wire (pts (xy 92.71 33.02) (xy 96.52 33.02))
     (stroke (width 0) (type default) (color 0 0 0 0))
@@
     (stroke (width 0) (type default) (color 0 0 0 0))
   )
-  (wire (pts (xy 49.53 25.4) (xy 53.34 25.4))
+  (wire (pts (xy 39.37 25.4) (xy 53.34 25.4))
     (stroke (width 0) (type default) (color 0 0 0 0))
   )
@@
     (effects (font (size 1.27 1.27)) (justify left bottom))
   )
+  (label "LIGHTGATE" (at 217.17 111.76 0)
+    (effects (font (size 1.27 1.27)) (justify left bottom))
+  )
   (label "PROG3V3" (at 231.14 82.55 0)
     (effects (font (size 1.27 1.27)) (justify left bottom))
@@
     (effects (font (size 1.27 1.27)) (justify left bottom))
   )
+  (label "LIGHTGATE" (at 146.05 163.83 0)
+    (effects (font (size 1.27 1.27)) (justify left bottom))
+  )
   (symbol (lib_id "74xx:CD74HC4067SM") (at 46.99 72.39 90) (unit 1)
     (in_bom yes) (on_board yes) (fields_autoplaced)
@@
   (symbol (lib_id "Connector:Conn_01x02_Female") (at 24.13 152.4 180) (unit 1)
     (in_bom yes) (on_board yes) (fields_autoplaced)
-    (property "Reference" "J5" (id 0) (at 24.765 144.78 0))
+    (property "Reference" "J4" (id 0) (at 24.765 144.78 0))
     (property "Value" "Conn_01x02_Female" (id 1) (at 24.765 147.32 0))
     (property "Footprint" "Connector_AMASS:AMASS_XT30UPB-F_1x02_P5.0mm_Vertical" (id 2) (at 24.13 152.4 0)
@@
     (pin "1")
   )
+  (symbol (lib_id "power:+5V") (at 146.05 151.13 270) (unit 1)
+    (in_bom yes) (on_board yes) (fields_autoplaced)
+    (property "Reference" "#PWR0106" (id 0) (at 142.24 151.13 0)
+      (effects (font (size 1.27 1.27)) hide)
+    )
+    (property "Value" "+5V" (id 1) (at 149.86 151.1299 90)
+      (effects (font (size 1.27 1.27)) (justify left))
+    )
+    (property "Footprint" "" (id 2) (at 146.05 151.13 0)
+      (effects (font (size 1.27 1.27)) hide)
+    )
+    (property "Datasheet" "" (id 3) (at 146.05 151.13 0)
+      (effects (font (size 1.27 1.27)) hide)
+    )
+    (pin "1")
+  )
   (symbol (lib_id "Switch:SW_Push") (at 252.73 161.29 0) (unit 1)
     (in_bom yes) (on_board yes) (fields_autoplaced)
@@
   (symbol (lib_id "Connector:Conn_01x03_Female") (at 24.13 120.65 180) (unit 1)
     (in_bom yes) (on_board yes) (fields_autoplaced)
-    (property "Reference" "J4" (id 0) (at 24.765 113.03 0))
-    (property "Value" "Conn_01x03_Female" (id 1) (at 24.765 115.57 0))
+    (property "Reference" "J3" (id 0) (at 24.765 113.03 0))
+    (property "Value" "DEBUG" (id 1) (at 24.765 115.57 0))
     (property "Footprint" "Connector_PinHeader_2.54mm:PinHeader_1x03_P2.54mm_Vertical" (id 2) (at 24.13 120.65 0)
       (effects (font (size 1.27 1.27)) hide)
@@
     (pin "2")
   )
+  (symbol (lib_id "power:GND") (at 146.05 153.67 90) (unit 1)
+    (in_bom yes) (on_board yes) (fields_autoplaced)
+    (property "Reference" "#PWR0104" (id 0) (at 152.4 153.67 0)
+      (effects (font (size 1.27 1.27)) hide)
+    )
+    (property "Value" "GND" (id 1) (at 149.86 153.6699 90)
+      (effects (font (size 1.27 1.27)) (justify right))
+    )
+    (property "Footprint" "" (id 2) (at 146.05 153.67 0)
+      (effects (font (size 1.27 1.27)) hide)
+    )
+    (property "Datasheet" "" (id 3) (at 146.05 153.67 0)
+      (effects (font (size 1.27 1.27)) hide)
+    )
+    (pin "1")
+  )
   (symbol (lib_id "Device:R_Photo") (at 134.62 55.88 0) (unit 1)
     (in_bom yes) (on_board yes) (fields_autoplaced)
@@
     (pin "2")
   )
+  (symbol (lib_id "power:VCCQ") (at 146.05 161.29 270) (unit 1)
+    (in_bom yes) (on_board yes) (fields_autoplaced)
+    (property "Reference" "#PWR0107" (id 0) (at 142.24 161.29 0)
+      (effects (font (size 1.27 1.27)) hide)
+    )
+    (property "Value" "VCCQ" (id 1) (at 149.86 161.2899 90)
+      (effects (font (size 1.27 1.27)) (justify left))
+    )
+    (property "Footprint" "" (id 2) (at 146.05 161.29 0)
+      (effects (font (size 1.27 1.27)) hide)
+    )
+    (property "Datasheet" "" (id 3) (at 146.05 161.29 0)
+      (effects (font (size 1.27 1.27)) hide)
+    )
+    (pin "1")
+  )
   (symbol (lib_id "power:GNDA") (at 228.6 64.77 90) (unit 1)
     (in_bom yes) (on_board yes) (fields_autoplaced)
@@
     (pin "2")
   )
+  (symbol (lib_id "Connector:Conn_01x02_Male") (at 140.97 151.13 0) (unit 1)
+    (in_bom yes) (on_board yes) (fields_autoplaced)
+    (property "Reference" "J5" (id 0) (at 141.605 146.05 0))
+    (property "Value" "Conn_01x02_Male" (id 1) (at 141.605 148.59 0))
+    (property "Footprint" "Connector_PinHeader_2.54mm:PinHeader_1x02_P2.54mm_Vertical" (id 2) (at 140.97 151.13 0)
+      (effects (font (size 1.27 1.27)) hide)
+    )
+    (property "Datasheet" "~" (id 3) (at 140.97 151.13 0)
+      (effects (font (size 1.27 1.27)) hide)
+    )
+    (pin "1")
+    (pin "2")
+  )
   (symbol (lib_id "Device:R") (at 109.22 146.05 0) (unit 1)
     (in_bom yes) (on_board yes) (fields_autoplaced)
@@
     (pin "9")
   )
-  (symbol (lib_id "Device:R") (at 45.72 25.4 90) (unit 1)
-    (in_bom yes) (on_board yes) (fields_autoplaced)
-    (property "Reference" "R33" (id 0) (at 45.72 19.05 90))
-    (property "Value" "0.39" (id 1) (at 45.72 21.59 90))
-    (property "Footprint" "Resistor_SMD:R_0603_1608Metric" (id 2) (at 45.72 27.178 90)
-      (effects (font (size 1.27 1.27)) hide)
-    )
-    (property "Datasheet" "~" (id 3) (at 45.72 25.4 0)
-      (effects (font (size 1.27 1.27)) hide)
-    )
-    (pin "1")
-    (pin "2")
-  )
   (symbol (lib_id "Device:LED") (at 88.9 29.21 90) (unit 1)
     (in_bom yes) (on_board yes) (fields_autoplaced)
@@
     (pin "2")
   )
+  (symbol (lib_id "Connector:Conn_01x02_Male") (at 140.97 161.29 0) (unit 1)
+    (in_bom yes) (on_board yes) (fields_autoplaced)
+    (property "Reference" "J6" (id 0) (at 141.605 156.21 0))
+    (property "Value" "Conn_01x02_Male" (id 1) (at 141.605 158.75 0))
+    (property "Footprint" "Connector_PinHeader_2.54mm:PinHeader_1x02_P2.54mm_Vertical" (id 2) (at 140.97 161.29 0)
+      (effects (font (size 1.27 1.27)) hide)
+    )
+    (property "Datasheet" "~" (id 3) (at 140.97 161.29 0)
+      (effects (font (size 1.27 1.27)) hide)
+    )
+    (pin "1")
+    (pin "2")
+  )
   (symbol (lib_id "Device:C") (at 248.92 142.24 90) (unit 1)
     (in_bom yes) (on_board yes) (fields_autoplaced)
@@
       (reference "#PWR0103") (unit 1) (value "+3V3") (footprint "")
     )
+    (path "/96308e0c-b20e-437f-8e95-fb0ed8af251c"
+      (reference "#PWR0104") (unit 1) (value "GND") (footprint "")
+    )
     (path "/8ba4a965-2eba-4e08-9e15-4d58d42275fd"
       (reference "#PWR0105") (unit 1) (value "GND") (footprint "")
     )
+    (path "/7fa4ee2e-f321-4354-85e7-27200ce4e707"
+      (reference "#PWR0106") (unit 1) (value "+5V") (footprint "")
+    )
+    (path "/9c559d8d-eaeb-4038-a16d-5253165c7519"
+      (reference "#PWR0107") (unit 1) (value "VCCQ") (footprint "")
+    )
     (path "/ee008ec7-5fc9-464d-9c4e-134d12caadc8"
       (reference "C1") (unit 1) (value "1μF") (footprint "Capacitor_SMD:C_0603_1608Metric")
@@
     )
     (path "/86937535-1a00-4375-a966-feffacfd480e"
-      (reference "J4") (unit 1) (value "Conn_01x03_Female") (footprint "Connector_PinHeader_2.54mm:PinHeader_1x03_P2.54mm_Vertical")
+      (reference "J3") (unit 1) (value "DEBUG") (footprint "Connector_PinHeader_2.54mm:PinHeader_1x03_P2.54mm_Vertical")
     )
     (path "/71e27d42-31a1-4137-acf4-0f589857544d"
-      (reference "J5") (unit 1) (value "Conn_01x02_Female") (footprint "Connector_AMASS:AMASS_XT30UPB-F_1x02_P5.0mm_Vertical")
+      (reference "J4") (unit 1) (value "Conn_01x02_Female") (footprint "Connector_AMASS:AMASS_XT30UPB-F_1x02_P5.0mm_Vertical")
+    )
+    (path "/afa1d923-ae3a-455a-8d44-9534c33289bf"
+      (reference "J5") (unit 1) (value "Conn_01x02_Male") (footprint "Connector_PinHeader_2.54mm:PinHeader_1x02_P2.54mm_Vertical")
+    )
+    (path "/cdf9e086-9a06-4aa5-a8b1-b04362ac6885"
+      (reference "J6") (unit 1) (value "Conn_01x02_Male") (footprint "Connector_PinHeader_2.54mm:PinHeader_1x02_P2.54mm_Vertical")
     )
     (path "/321f573f-a657-4c38-803b-a27027c026fb"
@@
       (reference "R32") (unit 1) (value "ALS-PT19-315C") (footprint "Resistor_SMD:R_0603_1608Metric")
     )
-    (path "/ccf313e4-fd72-4a8d-8931-81667a4cf4bb"
-      (reference "R33") (unit 1) (value "0.39") (footprint "Resistor_SMD:R_0603_1608Metric")
-    )
     (path "/e782a51f-adfb-46f6-b47e-41277c988231"

Commit message: submit all pcbs for production
Parts:
- added R33: 4.7k, Resistor_SMD:R_0603_1608Metric, symbol Device:R
Connections:
- net GND: no longer C2.2, C3.2, R34.2, R35.2, R36.2, R37.2, U2.12 (GND), U3.12 (GND)
- net GNDA: now also C2.2, C3.2, R34.2, R35.2, R36.2, R37.2, U2.12 (GND), U3.12 (GND), R33.2
- net LIGHTGATE: now also R33.1
Changed lines of the file:
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@@
     (stroke (width 0) (type default) (color 0 0 0 0))
   )
+  (wire (pts (xy 146.05 163.83) (xy 158.115 163.83))
+    (stroke (width 0) (type default) (color 0 0 0 0))
+  )
   (wire (pts (xy 63.5 154.305) (xy 63.5 152.4))
     (stroke (width 0) (type default) (color 0 0 0 0))
@@
     (effects (font (size 1.27 1.27)) (justify left bottom))
   )
+  (label "LIGHTGATE" (at 146.05 163.83 0)
+    (effects (font (size 1.27 1.27)) (justify left bottom))
+  )
   (label "DEBUGRX" (at 231.14 77.47 0)
     (effects (font (size 1.27 1.27)) (justify left bottom))
@@
     (effects (font (size 1.27 1.27)) (justify left bottom))
   )
-  (label "LIGHTGATE" (at 146.05 163.83 0)
-    (effects (font (size 1.27 1.27)) (justify left bottom))
-  )
   (symbol (lib_id "74xx:CD74HC4067SM") (at 46.99 72.39 90) (unit 1)
     (in_bom yes) (on_board yes) (fields_autoplaced)
@@
     (pin "2")
   )
+  (symbol (lib_id "Device:R") (at 161.925 163.83 90) (unit 1)
+    (in_bom yes) (on_board yes) (fields_autoplaced)
+    (property "Reference" "R33" (id 0) (at 161.925 157.48 90))
+    (property "Value" "4.7k" (id 1) (at 161.925 160.02 90))
+    (property "Footprint" "Resistor_SMD:R_0603_1608Metric" (id 2) (at 161.925 165.608 90)
+      (effects (font (size 1.27 1.27)) hide)
+    )
+    (property "Datasheet" "~" (id 3) (at 161.925 163.83 0)
+      (effects (font (size 1.27 1.27)) hide)
+    )
+    (pin "1")
+    (pin "2")
+  )
   (symbol (lib_id "power:GND") (at 243.84 138.43 270) (unit 1)
     (in_bom yes) (on_board yes) (fields_autoplaced)
@@
     (pin "2")
   )
+  (symbol (lib_id "power:GNDA") (at 165.735 163.83 90) (unit 1)
+    (in_bom yes) (on_board yes) (fields_autoplaced)
+    (property "Reference" "#PWR0108" (id 0) (at 172.085 163.83 0)
+      (effects (font (size 1.27 1.27)) hide)
+    )
+    (property "Value" "GNDA" (id 1) (at 168.91 163.8299 90)
+      (effects (font (size 1.27 1.27)) (justify right))
+    )
+    (property "Footprint" "" (id 2) (at 165.735 163.83 0)
+      (effects (font (size 1.27 1.27)) hide)
+    )
+    (property "Datasheet" "" (id 3) (at 165.735 163.83 0)
+      (effects (font (size 1.27 1.27)) hide)
+    )
+    (pin "1")
+  )
   (symbol (lib_id "Connector:Conn_01x03_Female") (at 24.13 120.65 180) (unit 1)
     (in_bom yes) (on_board yes) (fields_autoplaced)
@@
     (pin "1")
   )
-  (symbol (lib_id "power:GND") (at 21.59 102.87 0) (unit 1)
-    (in_bom yes) (on_board yes) (fields_autoplaced)
-    (property "Reference" "#PWR05" (id 0) (at 21.59 109.22 0)
-      (effects (font (size 1.27 1.27)) hide)
-    )
-    (property "Value" "GND" (id 1) (at 21.59 107.95 0))
-    (property "Footprint" "" (id 2) (at 21.59 102.87 0)
-      (effects (font (size 1.27 1.27)) hide)
-    )
-    (property "Datasheet" "" (id 3) (at 21.59 102.87 0)
-      (effects (font (size 1.27 1.27)) hide)
-    )
-    (pin "1")
-  )
   (symbol (lib_id "Device:C") (at 189.23 54.61 90) (unit 1)
     (in_bom yes) (on_board yes) (fields_autoplaced)
@@
     (pin "1")
   )
-  (symbol (lib_id "power:GND") (at 88.9 102.87 0) (unit 1)
-    (in_bom yes) (on_board yes) (fields_autoplaced)
-    (property "Reference" "#PWR07" (id 0) (at 88.9 109.22 0)
-      (effects (font (size 1.27 1.27)) hide)
-    )
-    (property "Value" "GND" (id 1) (at 88.9 107.95 0))
-    (property "Footprint" "" (id 2) (at 88.9 102.87 0)
-      (effects (font (size 1.27 1.27)) hide)
-    )
-    (property "Datasheet" "" (id 3) (at 88.9 102.87 0)
-      (effects (font (size 1.27 1.27)) hide)
-    )
-    (pin "1")
-  )
   (symbol (lib_id "Device:R_Photo") (at 52.07 55.88 0) (unit 1)
     (in_bom yes) (on_board yes) (fields_autoplaced)
@@
     (pin "2")
   )
+  (symbol (lib_id "power:GNDA") (at 21.59 102.87 0) (unit 1)
+    (in_bom yes) (on_board yes) (fields_autoplaced)
+    (property "Reference" "#PWR?" (id 0) (at 21.59 109.22 0)
+      (effects (font (size 1.27 1.27)) hide)
+    )
+    (property "Value" "GNDA" (id 1) (at 21.59 107.95 0))
+    (property "Footprint" "" (id 2) (at 21.59 102.87 0)
+      (effects (font (size 1.27 1.27)) hide)
+    )
+    (property "Datasheet" "" (id 3) (at 21.59 102.87 0)
+      (effects (font (size 1.27 1.27)) hide)
+    )
+    (pin "1")
+  )
   (symbol (lib_id "Device:LED") (at 138.43 29.21 90) (unit 1)
     (in_bom yes) (on_board yes) (fields_autoplaced)
@@
     (pin "2")
   )
+  (symbol (lib_id "power:GNDA") (at 88.9 102.87 0) (unit 1)
+    (in_bom yes) (on_board yes) (fields_autoplaced)
+    (property "Reference" "#PWR?" (id 0) (at 88.9 109.22 0)
+      (effects (font (size 1.27 1.27)) hide)
+    )
+    (property "Value" "GNDA" (id 1) (at 88.9 107.95 0))
+    (property "Footprint" "" (id 2) (at 88.9 102.87 0)
+      (effects (font (size 1.27 1.27)) hide)
+    )
+    (property "Datasheet" "" (id 3) (at 88.9 102.87 0)
+      (effects (font (size 1.27 1.27)) hide)
+    )
+    (pin "1")
+  )
   (symbol (lib_id "Switch:SW_DPDT_x2") (at 34.29 25.4 180) (unit 1)
     (in_bom yes) (on_board yes) (fields_autoplaced)
@@
       (reference "#PWR04") (unit 1) (value "+3V3") (footprint "")
     )
-    (path "/894d5f42-93e5-420f-bdd8-a122a9592963"
-      (reference "#PWR05") (unit 1) (value "GND") (footprint "")
-    )
     (path "/bec8aa97-af2d-4022-ae2a-233179caf957"
       (reference "#PWR06") (unit 1) (value "+3V3") (footprint "")
     )
-    (path "/c0f2b3eb-edde-496a-a44c-81a7a1e87d25"
-      (reference "#PWR07") (unit 1) (value "GND") (footprint "")
-    )
     (path "/b7166790-8d1d-4796-ad3e-76a1e1d84c69"
       (reference "#PWR08") (unit 1) (value "VCCQ") (footprint "")
@@
       (reference "#PWR0107") (unit 1) (value "VCCQ") (footprint "")
     )
+    (path "/866575c2-9c5e-4961-97ec-563dd5a98162"
+      (reference "#PWR0108") (unit 1) (value "GNDA") (footprint "")
+    )
+    (path "/d5b4b4d3-f70b-4265-a646-bae7623d2899"
+      (reference "#PWR?") (unit 1) (value "GNDA") (footprint "")
+    )
+    (path "/f27d1610-8a4d-4614-972c-2b4337aa0644"
+      (reference "#PWR?") (unit 1) (value "GNDA") (footprint "")
+    )
     (path "/ee008ec7-5fc9-464d-9c4e-134d12caadc8"
       (reference "C1") (unit 1) (value "1μF") (footprint "Capacitor_SMD:C_0603_1608Metric")
@@
       (reference "R32") (unit 1) (value "ALS-PT19-315C") (footprint "Resistor_SMD:R_0603_1608Metric")
     )
+    (path "/046e9cd3-2364-435f-8676-bf9f8bbd494d"
+      (reference "R33") (unit 1) (value "4.7k") (footprint "Resistor_SMD:R_0603_1608Metric")
+    )
     (path "/e782a51f-adfb-46f6-b47e-41277c988231"
