File: electrical design/layer3/layer3.kicad_sch (KiCad schematic)
At the start: 57 parts, among them J1 XT60PW-M, J10 SH1.0 Female, J11 SH1.0 Female, J12 MOTOR1, J13 MOTOR2, J14 MOTOR3, J15 MOTOR4, J16 CAMERA, J2 XT60PW-M, J3 XT30UPB-F, J4 XT30UPB-F, J5 XT30UPB-F, J6 XT30UPB-F, J7 XT30UPB-F, J8 COMPASS, J9 SH1.0 3P, SW1 SW_DPDT_x2, SW2 SW_Push, SW3 SW_DPDT_x2, SW4 SW_Push, U1 TEENSY 4.0, U2 STM32F103C8T6, U3 STM32F103C8T6, U4 74LVC2G04, U5 74LVC2G04, Y1 Crystal, Y2 Crystal

Commit message: almost final pcbs
Parts:
- removed J9: SH1.0 3P, Connector_JST:JST_SH_SM03B-SRSS-TB_1x03-1MP_P1.00mm_Horizontal, symbol Connector:Conn_01x03_Male
- added J17: SH1.0 3P, Connector_JST:JST_SH_BM03B-SRSS-TB_1x03-1MP_P1.00mm_Vertical, symbol Connector:Conn_01x03_Male
- added J9: SH1.0 5P, Connector_JST:JST_SH_BM05B-SRSS-TB_1x05-1MP_P1.00mm_Vertical, symbol Connector:Conn_01x05_Male
Connections:
- net +3V3: now also J9.4 (Pin_4)
- net +5V: now also J17.1 (Pin_1), J9.3 (Pin_3)
- net GND: now also J17.2 (Pin_2), J9.5 (Pin_5)
- net L1RX: now also J9.1 (Pin_1)
- net L1TX: now also J9.2 (Pin_2)
- net NEOPIXELOUT: now reaches U2.39 (PB3)
- net NEOPIXELOUT: now also J17.3 (Pin_3)
Changed lines of the file:
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@@
+    (effects (font (size 1.27 1.27)) (justify right bottom))
+  )
+  (label "L1RX" (at 76.2 147.32 0)
+    (effects (font (size 1.27 1.27)) (justify left bottom))
+  )
+  (label "NEOPIXELOUT" (at 129.54 118.11 180)
     (effects (font (size 1.27 1.27)) (justify right bottom))
   )
@@
     (effects (font (size 1.27 1.27)) (justify left bottom))
   )
+  (label "NEOPIXELOUT" (at 100.33 153.67 0)
+    (effects (font (size 1.27 1.27)) (justify left bottom))
+  )
   (label "LIDARRX" (at 33.02 115.57 0)
     (effects (font (size 1.27 1.27)) (justify left bottom))
@@
   )
   (label "BATT_+12V" (at 101.6 39.37 0)
+    (effects (font (size 1.27 1.27)) (justify left bottom))
+  )
+  (label "L1TX" (at 76.2 149.86 0)
     (effects (font (size 1.27 1.27)) (justify left bottom))
   )
@@
     (pin "1")
   )
+  (symbol (lib_id "power:GND") (at 76.2 157.48 90) (unit 1)
+    (in_bom yes) (on_board yes) (fields_autoplaced)
+    (property "Reference" "#PWR0129" (id 0) (at 82.55 157.48 0)
+      (effects (font (size 1.27 1.27)) hide)
+    )
+    (property "Value" "GND" (id 1) (at 80.01 157.4799 90)
+      (effects (font (size 1.27 1.27)) (justify right))
+    )
+    (property "Footprint" "" (id 2) (at 76.2 157.48 0)
+      (effects (font (size 1.27 1.27)) hide)
+    )
+    (property "Datasheet" "" (id 3) (at 76.2 157.48 0)
+      (effects (font (size 1.27 1.27)) hide)
+    )
+    (pin "1")
+  )
+  (symbol (lib_id "power:+3V3") (at 76.2 154.94 270) (unit 1)
+    (in_bom yes) (on_board yes) (fields_autoplaced)
+    (property "Reference" "#PWR0128" (id 0) (at 72.39 154.94 0)
+      (effects (font (size 1.27 1.27)) hide)
+    )
+    (property "Value" "+3V3" (id 1) (at 80.01 154.9399 90)
+      (effects (font (size 1.27 1.27)) (justify left))
+    )
+    (property "Footprint" "" (id 2) (at 76.2 154.94 0)
+      (effects (font (size 1.27 1.27)) hide)
+    )
+    (property "Datasheet" "" (id 3) (at 76.2 154.94 0)
+      (effects (font (size 1.27 1.27)) hide)
+    )
+    (pin "1")
+  )
   (symbol (lib_id "power:+3V3") (at 29.21 184.15 270) (unit 1)
     (in_bom yes) (on_board yes) (fields_autoplaced)
@@
     )
     (property "Datasheet" "" (id 3) (at 80.01 105.41 0)
+      (effects (font (size 1.27 1.27)) hide)
+    )
+    (pin "1")
+  )
+  (symbol (lib_id "power:GND") (at 100.33 151.13 90) (unit 1)
+    (in_bom yes) (on_board yes) (fields_autoplaced)
+    (property "Reference" "#PWR0130" (id 0) (at 106.68 151.13 0)
+      (effects (font (size 1.27 1.27)) hide)
+    )
+    (property "Value" "GND" (id 1) (at 104.14 151.1299 90)
+      (effects (font (size 1.27 1.27)) (justify right))
+    )
+    (property "Footprint" "" (id 2) (at 100.33 151.13 0)
+      (effects (font (size 1.27 1.27)) hide)
+    )
+    (property "Datasheet" "" (id 3) (at 100.33 151.13 0)
       (effects (font (size 1.27 1.27)) hide)
     )
@@
     (pin "1")
   )
+  (symbol (lib_id "Connector:Conn_01x03_Male") (at 95.25 151.13 0) (unit 1)
+    (in_bom yes) (on_board yes) (fields_autoplaced)
+    (property "Reference" "J17" (id 0) (at 95.885 143.51 0))
+    (property "Value" "SH1.0 3P" (id 1) (at 95.885 146.05 0))
+    (property "Footprint" "Connector_JST:JST_SH_BM03B-SRSS-TB_1x03-1MP_P1.00mm_Vertical" (id 2) (at 95.25 151.13 0)
+      (effects (font (size 1.27 1.27)) hide)
+    )
+    (property "Datasheet" "~" (id 3) (at 95.25 151.13 0)
+      (effects (font (size 1.27 1.27)) hide)
+    )
+    (pin "1")
+    (pin "2")
+    (pin "3")
+  )
   (symbol (lib_id "power:GND") (at 24.13 95.25 270) (unit 1)
     (in_bom yes) (on_board yes) (fields_autoplaced)
@@
     )
     (property "Datasheet" "" (id 3) (at 73.66 33.02 0)
+      (effects (font (size 1.27 1.27)) hide)
+    )
+    (pin "1")
+  )
+  (symbol (lib_id "power:+5V") (at 100.33 148.59 270) (unit 1)
+    (in_bom yes) (on_board yes) (fields_autoplaced)
+    (property "Reference" "#PWR0131" (id 0) (at 96.52 148.59 0)
+      (effects (font (size 1.27 1.27)) hide)
+    )
+    (property "Value" "+5V" (id 1) (at 104.14 148.5899 90)
+      (effects (font (size 1.27 1.27)) (justify left))
+    )
+    (property "Footprint" "" (id 2) (at 100.33 148.59 0)
+      (effects (font (size 1.27 1.27)) hide)
+    )
+    (property "Datasheet" "" (id 3) (at 100.33 148.59 0)
       (effects (font (size 1.27 1.27)) hide)
     )
@@
     (pin "1")
   )
+  (symbol (lib_id "power:+5V") (at 76.2 152.4 270) (unit 1)
+    (in_bom yes) (on_board yes) (fields_autoplaced)
+    (property "Reference" "#PWR0127" (id 0) (at 72.39 152.4 0)
+      (effects (font (size 1.27 1.27)) hide)
+    )
+    (property "Value" "+5V" (id 1) (at 80.01 152.3999 90)
+      (effects (font (size 1.27 1.27)) (justify left))
+    )
+    (property "Footprint" "" (id 2) (at 76.2 152.4 0)
+      (effects (font (size 1.27 1.27)) hide)
+    )
+    (property "Datasheet" "" (id 3) (at 76.2 152.4 0)
+      (effects (font (size 1.27 1.27)) hide)
+    )
+    (pin "1")
+  )
   (symbol (lib_id "power:+5V") (at 33.02 110.49 270) (unit 1)
     (in_bom yes) (on_board yes) (fields_autoplaced)
@@
     (pin "2")
   )
+  (symbol (lib_id "Connector:Conn_01x05_Male") (at 71.12 152.4 0) (unit 1)
+    (in_bom yes) (on_board yes) (fields_autoplaced)
+    (property "Reference" "J9" (id 0) (at 71.755 142.24 0))
+    (property "Value" "SH1.0 5P" (id 1) (at 71.755 144.78 0))
+    (property "Footprint" "Connector_JST:JST_SH_BM05B-SRSS-TB_1x05-1MP_P1.00mm_Vertical" (id 2) (at 71.12 152.4 0)
+      (effects (font (size 1.27 1.27)) hide)
+    )
+    (property "Datasheet" "~" (id 3) (at 71.12 152.4 0)
+      (effects (font (size 1.27 1.27)) hide)
+    )
+    (pin "1")
+    (pin "2")
+    (pin "3")
+    (pin "4")
+    (pin "5")
+  )
   (symbol (lib_id "Device:R") (at 269.24 30.48 90) (unit 1)
     (in_bom yes) (on_board yes)
@@
     )
     (pin "1")
-  )
-  (symbol (lib_id "Connector:Conn_01x03_Male") (at 71.12 149.86 0) (unit 1)
-    (in_bom yes) (on_board yes) (fields_autoplaced)
-    (property "Reference" "J9" (id 0) (at 71.755 142.24 0))
-    (property "Value" "SH1.0 3P" (id 1) (at 71.755 144.78 0))
-    (property "Footprint" "Connector_JST:JST_SH_SM03B-SRSS-TB_1x03-1MP_P1.00mm_Horizontal" (id 2) (at 71.12 149.86 0)
-      (effects (font (size 1.27 1.27)) hide)
-    )
-    (property "Datasheet" "~" (id 3) (at 71.12 149.86 0)
-      (effects (font (size 1.27 1.27)) hide)
-    )
-    (pin "1")
-    (pin "2")
-    (pin "3")
   )
   (symbol (lib_id "Connector:Conn_01x06_Female") (at 265.43 93.98 180) (unit 1)
@@
       (reference "#PWR0126") (unit 1) (value "+12V") (footprint "")
     )
+    (path "/99cb0b1e-6999-41d6-b50f-0bb0f2fda80a"
+      (reference "#PWR0127") (unit 1) (value "+5V") (footprint "")
+    )
+    (path "/20240fa3-7ce8-40d7-a2f1-97917f11fbcb"
+      (reference "#PWR0128") (unit 1) (value "+3V3") (footprint "")
+    )
+    (path "/1e2cc2f7-f086-4909-98cf-b105b573cb1a"
+      (reference "#PWR0129") (unit 1) (value "GND") (footprint "")
+    )
+    (path "/2a5b6097-a810-4911-abc0-8bb7d9ff9a42"
+      (reference "#PWR0130") (unit 1) (value "GND") (footprint "")
+    )
+    (path "/698ac68a-f83f-4a41-bccb-2077502f2578"
+      (reference "#PWR0131") (unit 1) (value "+5V") (footprint "")
+    )
     (path "/05568742-0152-4de6-b990-21dd9f504cc9"
       (reference "BT1") (unit 1) (value "Conn_01x06_Female") (footprint "Connector_PinSocket_2.54mm:PinSocket_1x06_P2.54mm_Horizontal")
@@
       (reference "J8") (unit 1) (value "COMPASS") (footprint "Connector_PinHeader_2.54mm:PinHeader_1x06_P2.54mm_Vertical")
     )
-    (path "/ec68e339-0b7d-4cf2-a98c-97c054e1c70a"
-      (reference "J9") (unit 1) (value "SH1.0 3P") (footprint "Connector_JST:JST_SH_SM03B-SRSS-TB_1x03-1MP_P1.00mm_Horizontal")
+    (path "/daca1efc-a3bf-4452-8f59-ca40e567f22f"
+      (reference "J9") (unit 1) (value "SH1.0 5P") (footprint "Connector_JST:JST_SH_BM05B-SRSS-TB_1x05-1MP_P1.00mm_Vertical")
     )
     (path "/2be1ad09-ec0a-4cb3-9b55-1fe07d2b63e8"
@@
       (reference "J16") (unit 1) (value "CAMERA") (footprint "Connector_JST:JST_GH_SM06B-GHS-TB_1x06-1MP_P1.25mm_Horizontal")
     )
+    (path "/659b9d32-8c23-423e-ae86-95604841f776"
+      (reference "J17") (unit 1) (value "SH1.0 3P") (footprint "Connector_JST:JST_SH_BM03B-SRSS-TB_1x03-1MP_P1.00mm_Vertical")
+    )
     (path "/9300e5e2-5178-4c12-b469-7b3a3947df1e"

Commit message: submit all pcbs for production
Parts:
- added J18: XT30UPB-F, Connector_AMASS:AMASS_XT30UPB-F_1x02_P5.0mm_Vertical, symbol Connector:Conn_01x02_Female
- added J19, J20: Conn_01x01_Female, Connector_Wire:SolderWire-1.5sqmm_1x01_D1.7mm_OD3.9mm, symbol Connector:Conn_01x01_Female
Connections:
- net MCU3V3 is gone; now on net MCU3V32: J8.1 (Pin_1), R1.2, R2.2
- net +12V: now also J2.2 (Pin_2); no longer J2.1 (Pin_1), J7.2 (Pin_2)
- net BATT_+12V: now also J2.1 (Pin_1), J7.2 (Pin_2), J18.2 (Pin_2), J19.1 (Pin_1), J20.1 (Pin_1); no longer J2.2 (Pin_2)
- net GND: now also J18.1 (Pin_1)
Changed lines of the file:
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@@
   (title_block
     (title "layer 3 schematic drawing")
-    (date "2023-01-29")
-    (rev "0.5")
+    (date "2023-02-15")
+    (rev "1.0")
     (company "8076 Robotics")
   )
@@
     (effects (font (size 1.27 1.27)) (justify right bottom))
   )
+  (label "BATT_+12V" (at 80.01 113.03 180)
+    (effects (font (size 1.27 1.27)) (justify right bottom))
+  )
+  (label "BATT_+12V" (at 115.57 168.91 180)
+    (effects (font (size 1.27 1.27)) (justify right bottom))
+  )
   (label "L1RX" (at 76.2 147.32 0)
     (effects (font (size 1.27 1.27)) (justify left bottom))
@@
     (effects (font (size 1.27 1.27)) (justify left bottom))
   )
+  (label "BATT_+12V" (at 101.6 49.53 0)
+    (effects (font (size 1.27 1.27)) (justify left bottom))
+  )
   (label "BATT_+12V" (at 27.94 85.09 180)
     (effects (font (size 1.27 1.27)) (justify right bottom))
@@
     (effects (font (size 1.27 1.27)) (justify left bottom))
   )
-  (label "MCU3V3" (at 86.36 116.205 270)
+  (label "MCU3V32" (at 86.36 116.205 270)
     (effects (font (size 1.27 1.27)) (justify right bottom))
   )
@@
     (effects (font (size 1.27 1.27)) (justify left bottom))
   )
+  (label "BATT_+12V" (at 115.57 175.26 180)
+    (effects (font (size 1.27 1.27)) (justify right bottom))
+  )
   (label "SWDIO1" (at 162.56 143.51 0)
     (effects (font (size 1.27 1.27)) (justify left bottom))
@@
     (effects (font (size 1.27 1.27)) (justify left bottom))
   )
+  (label "BATT_+12V" (at 115.57 181.61 180)
+    (effects (font (size 1.27 1.27)) (justify right bottom))
+  )
   (label "SWDIO1" (at 176.53 93.98 0)
     (effects (font (size 1.27 1.27)) (justify left bottom))
@@
     (effects (font (size 1.27 1.27)) (justify left bottom))
   )
-  (label "BATT_+12V" (at 101.6 52.07 0)
-    (effects (font (size 1.27 1.27)) (justify left bottom))
-  )
   (symbol (lib_id "Connector:Conn_01x06_Female") (at 33.02 95.25 0) (unit 1)
     (in_bom yes) (on_board yes) (fields_autoplaced)
@@
     (pin "1")
   )
+  (symbol (lib_id "Connector:Conn_01x01_Female") (at 120.65 175.26 0) (unit 1)
+    (in_bom yes) (on_board yes) (fields_autoplaced)
+    (property "Reference" "J19" (id 0) (at 121.92 173.9899 0)
+      (effects (font (size 1.27 1.27)) (justify left))
+    )
+    (property "Value" "Conn_01x01_Female" (id 1) (at 121.92 176.5299 0)
+      (effects (font (size 1.27 1.27)) (justify left))
+    )
+    (property "Footprint" "Connector_Wire:SolderWire-1.5sqmm_1x01_D1.7mm_OD3.9mm" (id 2) (at 120.65 175.26 0)
+      (effects (font (size 1.27 1.27)) hide)
+    )
+    (property "Datasheet" "~" (id 3) (at 120.65 175.26 0)
+      (effects (font (size 1.27 1.27)) hide)
+    )
+    (pin "1")
+  )
   (symbol (lib_id "Connector:Conn_01x06_Female") (at 171.45 93.98 180) (unit 1)
     (in_bom yes) (on_board yes) (fields_autoplaced)
@@
     (pin "1")
   )
+  (symbol (lib_id "Connector:Conn_01x02_Female") (at 120.65 166.37 0) (unit 1)
+    (in_bom yes) (on_board yes) (fields_autoplaced)
+    (property "Reference" "J18" (id 0) (at 121.92 166.3699 0)
+      (effects (font (size 1.27 1.27)) (justify left))
+    )
+    (property "Value" "XT30UPB-F" (id 1) (at 121.92 168.9099 0)
+      (effects (font (size 1.27 1.27)) (justify left))
+    )
+    (property "Footprint" "Connector_AMASS:AMASS_XT30UPB-F_1x02_P5.0mm_Vertical" (id 2) (at 120.65 166.37 0)
+      (effects (font (size 1.27 1.27)) hide)
+    )
+    (property "Datasheet" "~" (id 3) (at 120.65 166.37 0)
+      (effects (font (size 1.27 1.27)) hide)
+    )
+    (pin "1")
+    (pin "2")
+  )
   (symbol (lib_id "power:+3V3") (at 73.66 66.04 270) (unit 1)
     (in_bom yes) (on_board yes) (fields_autoplaced)
@@
     (pin "1")
   )
+  (symbol (lib_id "Connector:Conn_01x01_Female") (at 120.65 181.61 0) (unit 1)
+    (in_bom yes) (on_board yes) (fields_autoplaced)
+    (property "Reference" "J20" (id 0) (at 121.92 180.3399 0)
+      (effects (font (size 1.27 1.27)) (justify left))
+    )
+    (property "Value" "Conn_01x01_Female" (id 1) (at 121.92 182.8799 0)
+      (effects (font (size 1.27 1.27)) (justify left))
+    )
+    (property "Footprint" "Connector_Wire:SolderWire-1.5sqmm_1x01_D1.7mm_OD3.9mm" (id 2) (at 120.65 181.61 0)
+      (effects (font (size 1.27 1.27)) hide)
+    )
+    (property "Datasheet" "~" (id 3) (at 120.65 181.61 0)
+      (effects (font (size 1.27 1.27)) hide)
+    )
+    (pin "1")
+  )
   (symbol (lib_id "power:GND") (at 73.66 30.48 90) (unit 1)
     (in_bom yes) (on_board yes) (fields_autoplaced)
@@
     (pin "2")
   )
-  (symbol (lib_id "power:+12V") (at 101.6 49.53 270) (unit 1)
-    (in_bom yes) (on_board yes) (fields_autoplaced)
-    (property "Reference" "#PWR0108" (id 0) (at 97.79 49.53 0)
-      (effects (font (size 1.27 1.27)) hide)
-    )
-    (property "Value" "+12V" (id 1) (at 105.41 49.5299 90)
-      (effects (font (size 1.27 1.27)) (justify left))
-    )
-    (property "Footprint" "" (id 2) (at 101.6 49.53 0)
-      (effects (font (size 1.27 1.27)) hide)
-    )
-    (property "Datasheet" "" (id 3) (at 101.6 49.53 0)
-      (effects (font (size 1.27 1.27)) hide)
-    )
-    (pin "1")
-  )
   (symbol (lib_id "power:+3V3") (at 45.72 184.15 270) (unit 1)
     (in_bom yes) (on_board yes) (fields_autoplaced)
@@
     (pin "2")
   )
-  (symbol (lib_id "power:+12V") (at 80.01 113.03 90) (unit 1)
-    (in_bom yes) (on_board yes) (fields_autoplaced)
-    (property "Reference" "#PWR0126" (id 0) (at 83.82 113.03 0)
-      (effects (font (size 1.27 1.27)) hide)
-    )
-    (property "Value" "+12V" (id 1) (at 76.2 113.0299 90)
-      (effects (font (size 1.27 1.27)) (justify left))
-    )
-    (property "Footprint" "" (id 2) (at 80.01 113.03 0)
-      (effects (font (size 1.27 1.27)) hide)
-    )
-    (property "Datasheet" "" (id 3) (at 80.01 113.03 0)
-      (effects (font (size 1.27 1.27)) hide)
-    )
-    (pin "1")
-  )
   (symbol (lib_id "power:GND") (at 231.14 30.48 270) (unit 1)
     (in_bom yes) (on_board yes) (fields_autoplaced)
@@
     (pin "1")
   )
+  (symbol (lib_id "power:+12V") (at 101.6 52.07 270) (unit 1)
+    (in_bom yes) (on_board yes) (fields_autoplaced)
+    (property "Reference" "#PWR0108" (id 0) (at 97.79 52.07 0)
+      (effects (font (size 1.27 1.27)) hide)
+    )
+    (property "Value" "+12V" (id 1) (at 105.41 52.0699 90)
+      (effects (font (size 1.27 1.27)) (justify left))
+    )
+    (property "Footprint" "" (id 2) (at 101.6 52.07 0)
+      (effects (font (size 1.27 1.27)) hide)
+    )
+    (property "Datasheet" "" (id 3) (at 101.6 52.07 0)
+      (effects (font (size 1.27 1.27)) hide)
+    )
+    (pin "1")
+  )
   (symbol (lib_id "Device:C") (at 201.93 52.07 90) (unit 1)
     (in_bom yes) (on_board yes) (fields_autoplaced)
@@
     (pin "1")
   )
+  (symbol (lib_id "power:GND") (at 115.57 166.37 270) (unit 1)
+    (in_bom yes) (on_board yes) (fields_autoplaced)
+    (property "Reference" "#PWR0133" (id 0) (at 109.22 166.37 0)
+      (effects (font (size 1.27 1.27)) hide)
+    )
+    (property "Value" "GND" (id 1) (at 111.76 166.3699 90)
+      (effects (font (size 1.27 1.27)) (justify right))
+    )
+    (property "Footprint" "" (id 2) (at 115.57 166.37 0)
+      (effects (font (size 1.27 1.27)) hide)
+    )
+    (property "Datasheet" "" (id 3) (at 115.57 166.37 0)
+      (effects (font (size 1.27 1.27)) hide)
+    )
+    (pin "1")
+  )
   (symbol (lib_id "Connector:Conn_01x03_Female") (at 55.88 82.55 0) (unit 1)
     (in_bom yes) (on_board yes) (fields_autoplaced)
@@
       (reference "#PWR0107") (unit 1) (value "+5V") (footprint "")
     )
-    (path "/80fd3eb9-7ad4-41f8-a7f1-19ecc30e10a7"
+    (path "/c83c0645-7b3f-4f6d-bed2-191f6b4b1886"
       (reference "#PWR0108") (unit 1) (value "+12V") (footprint "")
     )
@@
       (reference "#PWR0125") (unit 1) (value "+5V") (footprint "")
     )
-    (path "/a88bb7bc-96f2-4209-8a91-29a0ff561a0b"
-      (reference "#PWR0126") (unit 1) (value "+12V") (footprint "")
-    )
     (path "/99cb0b1e-6999-41d6-b50f-0bb0f2fda80a"
       (reference "#PWR0127") (unit 1) (value "+5V") (footprint "")
@@
       (reference "#PWR0131") (unit 1) (value "+5V") (footprint "")
     )
+    (path "/d3ae9d65-df68-4008-a4c6-402b581ba7a9"
+      (reference "#PWR0133") (unit 1) (value "GND") (footprint "")
+    )
     (path "/05568742-0152-4de6-b990-21dd9f504cc9"
       (reference "BT1") (unit 1) (value "Conn_01x06_Female") (footprint "Connector_PinSocket_2.54mm:PinSocket_1x06_P2.54mm_Horizontal")
@@
       (reference "J17") (unit 1) (value "SH1.0 3P") (footprint "Connector_JST:JST_SH_BM03B-SRSS-TB_1x03-1MP_P1.00mm_Vertical")
     )
+    (path "/3214d8c1-e52a-48ab-8c31-5dc0c17687f0"
+      (reference "J18") (unit 1) (value "XT30UPB-F") (footprint "Connector_AMASS:AMASS_XT30UPB-F_1x02_P5.0mm_Vertical")
+    )
+    (path "/2a831ee9-8bbd-4948-911c-44926172527f"
+      (reference "J19") (unit 1) (value "Conn_01x01_Female") (footprint "Connector_Wire:SolderWire-1.5sqmm_1x01_D1.7mm_OD3.9mm")
+    )
+    (path "/5ce09a58-1c00-440b-b753-8e5051f0c9cc"
+      (reference "J20") (unit 1) (value "Conn_01x01_Female") (footprint "Connector_Wire:SolderWire-1.5sqmm_1x01_D1.7mm_OD3.9mm")
+    )
     (path "/9300e5e2-5178-4c12-b469-7b3a3947df1e"
